File: PFD/Eagle/Motherboard/PFD Board.sch (EAGLE design)
At the start: 14 parts, among them IC1 MCP23017SO, SW1 1825910-6

Commit message: Corrected RESET switch design.
Parts:
- SW1: value 1825910-6 -> 3-1825910-1; device Switch:1825910-6 -> Switches:3-1825910-1
Changed lines of the file:
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@@
 <part name="R3" library="rcl" library_urn="urn:adsk.eagle:library:334" deviceset="R-EU_" device="0207/10" package3d_urn="urn:adsk.eagle:package:23491/2" value="4k7"/>
 <part name="R4" library="rcl" library_urn="urn:adsk.eagle:library:334" deviceset="R-EU_" device="0207/10" package3d_urn="urn:adsk.eagle:package:23491/2" value="4k7"/>
-<part name="SW1" library="Switch" library_urn="urn:adsk.eagle:library:11396471" deviceset="1825910-6" device="" package3d_urn="urn:adsk.eagle:package:12788209/4"/>
+<part name="SW1" library="Switches" library_urn="urn:adsk.eagle:library:14854419" deviceset="3-1825910-1" device="" package3d_urn="urn:adsk.eagle:package:14854625/2"/>
 <part name="C1" library="rcl" library_urn="urn:adsk.eagle:library:334" deviceset="C-EU" device="025-025X050" package3d_urn="urn:adsk.eagle:package:23629/2"/>
 <part name="C2" library="rcl" library_urn="urn:adsk.eagle:library:334" deviceset="CPOL-EU" device="E2.5-5" package3d_urn="urn:adsk.eagle:package:23344/1"/>
@@
 <attribute name="VALUE" x="-3.81" y="67.818" size="1.778" layer="96"/>
 </instance>
-<instance part="SW1" gate="G$1" x="91.44" y="43.18" smashed="yes">
+<instance part="SW1" gate="A" x="91.44" y="43.18" smashed="yes">
 <attribute name="NAME" x="86.3503" y="49.03315" size="1.803440625" layer="95"/>
 <attribute name="VALUE" x="86.351690625" y="35.54753125" size="1.802940625" layer="96"/>
@@
 </segment>
 <segment>
-<pinref part="SW1" gate="G$1" pin="3"/>
-<wire x1="101.6" y1="45.72" x2="106.68" y2="45.72" width="0.1524" layer="91"/>
+<pinref part="SW1" gate="A" pin="3"/>
+<wire x1="109.22" y1="45.72" x2="106.68" y2="45.72" width="0.1524" layer="91"/>
 <label x="101.6" y="45.72" size="1.778" layer="95"/>
 </segment>
@@
 <pinref part="B1" gate="G$1" pin="RESET"/>
 <label x="58.42" y="43.18" size="1.778" layer="95" align="bottom-right"/>
-<pinref part="SW1" gate="G$1" pin="1"/>
-<wire x1="81.28" y1="45.72" x2="81.28" y2="43.18" width="0.1524" layer="91"/>
+<pinref part="SW1" gate="A" pin="1"/>
+<wire x1="73.66" y1="45.72" x2="81.28" y2="43.18" width="0.1524" layer="91"/>
 <wire x1="81.28" y1="43.18" x2="48.26" y2="43.18" width="0.1524" layer="91"/>
 </segment>
@@
 <segment>
 <pinref part="R2" gate="G$1" pin="1"/>
-<pinref part="SW1" gate="G$1" pin="2"/>
-<wire x1="78.74" y1="40.64" x2="81.28" y2="40.64" width="0.1524" layer="91"/>
-</segment>
-</net>
+<pinref part="SW1" gate="A" pin="2"/>
+<wire x1="78.74" y1="40.64" x2="73.66" y2="38.1" width="0.1524" layer="91"/>
+</segment>
+</net>
